File: hardware/hardware.kicad_sch (KiCad schematic)
At the start: 71 parts, among them J1 USB_B, SW1 SW_POWER, U1 NE555P, U2 LM386, U3 LM3914V

Commit message: more schematics
Parts:
- added J2: AUDIO, Connector_Audio:Jack_3.5mm_Ledino_KB3SPRS_Horizontal, symbol Connector:AudioJack2
- added J3: STYLUS, Connector_Audio:Jack_3.5mm_Ledino_KB3SPRS_Horizontal, symbol Connector:AudioJack2
- J1: footprint (none) -> Connector_USB:USB_B_Lumberg_2411_02_Horizontal
- RV1, RV2, RV3, RV4, RV5: footprint Potentiometer_THT:Potentiometer_Piher_T-16L_Single_Vertical_Hole -> keyboard:potm
Connections:
- net AUDIO_OUT: now also J2.T
- net GND: now also J2.S
- net KB_IN: now also J3.S, J3.T
Other:
- note added: "stylus"
- moved on the sheet: RV5, TP11

Commit message: more hardware
Parts:
- U3: footprint Package_LCC:PLCC-20 -> keyboard:avans-lm3914v
- renumbered TP11 to TP1, TP22 to TP2
Other:
- note added: "TODO: - audio versterker afmaken - vu meter - stylus verbindingen - peak detector voor lm3914 vu meter - meer footprints toevoegen"
- note removed: "TODO: - audio versterker afmaken - vu meter - stylus verbindingen - peak detector voor lm3914 vu meter"
Changed lines of the file:
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@@
     (effects (font (size 1.27 1.27)) (justify left bottom))
   )
-  (text "TODO:\n- audio versterker afmaken\n- vu meter\n- stylus verbindingen\n- peak detector voor lm3914 vu meter"
+  (text "TODO:\n- audio versterker afmaken\n- vu meter\n- stylus verbindingen\n- peak detector voor lm3914 vu meter\n- meer footprints toevoegen"
     (at 13.97 196.215 0)
     (effects (font (size 1.27 1.27)) (justify left bottom))
@@
   (symbol (lib_id "power:GND") (at 27.94 41.275 0) (unit 1)
     (in_bom yes) (on_board yes) (fields_autoplaced)
-    (property "Reference" "#PWR012" (id 0) (at 27.94 47.625 0)
+    (property "Reference" "#PWR011" (id 0) (at 27.94 47.625 0)
       (effects (font (size 1.27 1.27)) hide)
     )
@@
   (symbol (lib_id "Connector:TestPoint") (at 41.91 125.095 270) (unit 1)
     (in_bom yes) (on_board yes) (fields_autoplaced)
-    (property "Reference" "TP22" (id 0) (at 47.625 123.8249 90)
+    (property "Reference" "TP2" (id 0) (at 47.625 123.8249 90)
       (effects (font (size 1.27 1.27)) (justify left))
     )
@@
   (symbol (lib_id "Connector:TestPoint_Probe") (at 231.14 80.645 270) (unit 1)
     (in_bom yes) (on_board yes)
-    (property "Reference" "TP11" (id 0) (at 228.6 86.995 90)
+    (property "Reference" "TP1" (id 0) (at 228.6 86.995 90)
       (effects (font (size 1.27 1.27)) (justify left))
     )
@@
   (symbol (lib_id "power:VCC") (at 109.22 75.565 0) (unit 1)
     (in_bom yes) (on_board yes)
-    (property "Reference" "#PWR021" (id 0) (at 109.22 79.375 0)
+    (property "Reference" "#PWR020" (id 0) (at 109.22 79.375 0)
       (effects (font (size 1.27 1.27)) hide)
     )
@@
   (symbol (lib_id "power:VCC") (at 44.45 69.85 0) (unit 1)
     (in_bom yes) (on_board yes) (fields_autoplaced)
-    (property "Reference" "#PWR020" (id 0) (at 44.45 73.66 0)
+    (property "Reference" "#PWR019" (id 0) (at 44.45 73.66 0)
       (effects (font (size 1.27 1.27)) hide)
     )
@@
   (symbol (lib_id "power:GND") (at 47.625 43.815 0) (unit 1)
     (in_bom yes) (on_board yes)
-    (property "Reference" "#PWR013" (id 0) (at 47.625 50.165 0)
+    (property "Reference" "#PWR012" (id 0) (at 47.625 50.165 0)
       (effects (font (size 1.27 1.27)) hide)
     )
@@
   (symbol (lib_id "power:GND") (at 177.165 78.74 0) (unit 1)
     (in_bom yes) (on_board yes) (fields_autoplaced)
-    (property "Reference" "#PWR010" (id 0) (at 177.165 85.09 0)
+    (property "Reference" "#PWR022" (id 0) (at 177.165 85.09 0)
       (effects (font (size 1.27 1.27)) hide)
     )
@@
   (symbol (lib_id "power:GND") (at 37.465 54.61 0) (unit 1)
     (in_bom yes) (on_board yes) (fields_autoplaced)
-    (property "Reference" "#PWR016" (id 0) (at 37.465 60.96 0)
+    (property "Reference" "#PWR015" (id 0) (at 37.465 60.96 0)
       (effects (font (size 1.27 1.27)) hide)
     )
@@
       (effects (font (size 1.27 1.27)) (justify left))
     )
-    (property "Footprint" "Package_LCC:PLCC-20" (id 2) (at 109.22 93.345 0)
+    (property "Footprint" "keyboard:avans-lm3914v" (id 2) (at 109.22 93.345 0)
       (effects (font (size 1.27 1.27)) hide)
     )
@@
   (symbol (lib_id "power:VCC") (at 214.63 67.31 0) (unit 1)
     (in_bom yes) (on_board yes)
-    (property "Reference" "#PWR019" (id 0) (at 214.63 71.12 0)
+    (property "Reference" "#PWR018" (id 0) (at 214.63 71.12 0)
       (effects (font (size 1.27 1.27)) hide)
     )
@@
   (symbol (lib_id "power:GND") (at 101.6 76.835 0) (unit 1)
     (in_bom yes) (on_board yes)
-    (property "Reference" "#PWR022" (id 0) (at 101.6 83.185 0)
+    (property "Reference" "#PWR021" (id 0) (at 101.6 83.185 0)
       (effects (font (size 1.27 1.27)) hide)
     )
@@
   (symbol (lib_id "power:GND") (at 144.78 67.31 0) (unit 1)
     (in_bom yes) (on_board yes)
-    (property "Reference" "#PWR018" (id 0) (at 144.78 73.66 0)
+    (property "Reference" "#PWR017" (id 0) (at 144.78 73.66 0)
       (effects (font (size 1.27 1.27)) hide)
     )
@@
   (symbol (lib_id "power:VCC") (at 152.4 66.04 0) (unit 1)
     (in_bom yes) (on_board yes)
-    (property "Reference" "#PWR017" (id 0) (at 152.4 69.85 0)
+    (property "Reference" "#PWR016" (id 0) (at 152.4 69.85 0)
       (effects (font (size 1.27 1.27)) hide)
     )
@@
   (symbol (lib_id "power:GND") (at 108.585 51.435 0) (unit 1)
     (in_bom yes) (on_board yes)
-    (property "Reference" "#PWR015" (id 0) (at 108.585 57.785 0)
+    (property "Reference" "#PWR014" (id 0) (at 108.585 57.785 0)
       (effects (font (size 1.27 1.27)) hide)
     )
@@
   (symbol (lib_id "power:GND") (at 234.95 48.26 0) (unit 1)
     (in_bom yes) (on_board yes) (fields_autoplaced)
-    (property "Reference" "#PWR014" (id 0) (at 234.95 54.61 0)
+    (property "Reference" "#PWR013" (id 0) (at 234.95 54.61 0)
       (effects (font (size 1.27 1.27)) hide)
     )
@@
   (symbol (lib_id "power:VCC") (at 34.925 38.735 0) (unit 1)
     (in_bom yes) (on_board yes)
-    (property "Reference" "#PWR011" (id 0) (at 34.925 42.545 0)
+    (property "Reference" "#PWR010" (id 0) (at 34.925 42.545 0)
       (effects (font (size 1.27 1.27)) hide)
     )
@@
       (reference "#PWR09") (unit 1) (value "GND") (footprint "")
     )
+    (path "/dcce6d87-e6b7-4840-a059-2bc2dbd30498"
+      (reference "#PWR010") (unit 1) (value "VCC") (footprint "")
+    )
+    (path "/15c38692-ed8d-47dc-bc28-8ed36b9df2dd"
+      (reference "#PWR011") (unit 1) (value "GND") (footprint "")
+    )
+    (path "/517aeb5d-8eab-4421-9d39-bacc4bae273d"
+      (reference "#PWR012") (unit 1) (value "GND") (footprint "")
+    )
+    (path "/d464a4cf-082d-41cd-8c3b-20e148aa391a"
+      (reference "#PWR013") (unit 1) (value "GND") (footprint "")
+    )
+    (path "/d2e5d02a-f21f-49ad-9b4d-48d42ccab4de"
+      (reference "#PWR014") (unit 1) (value "GND") (footprint "")
+    )
+    (path "/67b4ff9a-2ae2-4c62-b24d-b29a9b1ca1f1"
+      (reference "#PWR015") (unit 1) (value "GND") (footprint "")
+    )
+    (path "/cbe7e145-59d3-4ea1-b7b9-7b1a2d4b606a"
+      (reference "#PWR016") (unit 1) (value "VCC") (footprint "")
+    )
+    (path "/a9447a92-7db6-402e-bcea-df15e6e83fec"
+      (reference "#PWR017") (unit 1) (value "GND") (footprint "")
+    )
+    (path "/74303408-51a6-4ff7-bd06-96f2272bc939"
+      (reference "#PWR018") (unit 1) (value "VCC") (footprint "")
+    )
+    (path "/41568218-681a-410c-9bd0-ca60fb10f910"
+      (reference "#PWR019") (unit 1) (value "VCC") (footprint "")
+    )
+    (path "/32e35549-1494-475d-a291-f2e290cb592a"
+      (reference "#PWR020") (unit 1) (value "VCC") (footprint "")
+    )
+    (path "/87fc1511-4a34-41e1-99b9-d6d239f5984d"
+      (reference "#PWR021") (unit 1) (value "GND") (footprint "")
+    )
     (path "/598483d5-163b-475c-83a1-684fb184809e"
-      (reference "#PWR010") (unit 1) (value "GND") (footprint "")
-    )
-    (path "/dcce6d87-e6b7-4840-a059-2bc2dbd30498"
-      (reference "#PWR011") (unit 1) (value "VCC") (footprint "")
-    )
-    (path "/15c38692-ed8d-47dc-bc28-8ed36b9df2dd"
-      (reference "#PWR012") (unit 1) (value "GND") (footprint "")
-    )
-    (path "/517aeb5d-8eab-4421-9d39-bacc4bae273d"
-      (reference "#PWR013") (unit 1) (value "GND") (footprint "")
-    )
-    (path "/d464a4cf-082d-41cd-8c3b-20e148aa391a"
-      (reference "#PWR014") (unit 1) (value "GND") (footprint "")
-    )
-    (path "/d2e5d02a-f21f-49ad-9b4d-48d42ccab4de"
-      (reference "#PWR015") (unit 1) (value "GND") (footprint "")
-    )
-    (path "/67b4ff9a-2ae2-4c62-b24d-b29a9b1ca1f1"
-      (reference "#PWR016") (unit 1) (value "GND") (footprint "")
-    )
-    (path "/cbe7e145-59d3-4ea1-b7b9-7b1a2d4b606a"
-      (reference "#PWR017") (unit 1) (value "VCC") (footprint "")
-    )
-    (path "/a9447a92-7db6-402e-bcea-df15e6e83fec"
-      (reference "#PWR018") (unit 1) (value "GND") (footprint "")
-    )
-    (path "/74303408-51a6-4ff7-bd06-96f2272bc939"
-      (reference "#PWR019") (unit 1) (value "VCC") (footprint "")
-    )
-    (path "/41568218-681a-410c-9bd0-ca60fb10f910"
-      (reference "#PWR020") (unit 1) (value "VCC") (footprint "")
-    )
-    (path "/32e35549-1494-475d-a291-f2e290cb592a"
-      (reference "#PWR021") (unit 1) (value "VCC") (footprint "")
-    )
-    (path "/87fc1511-4a34-41e1-99b9-d6d239f5984d"
       (reference "#PWR022") (unit 1) (value "GND") (footprint "")
     )
@@
     )
     (path "/32454f40-aaf4-4cba-98e8-18cd94593c9e"
-      (reference "TP11") (unit 1) (value "STYLUS") (footprint "")
+      (reference "TP1") (unit 1) (value "STYLUS") (footprint "")
     )
     (path "/16bc0c8a-1942-4688-b8e3-caef7378a407"
-      (reference "TP22") (unit 1) (value "REF_GND") (footprint "")
+      (reference "TP2") (unit 1) (value "REF_GND") (footprint "")
     )
     (path "/f554789c-667d-4105-98f7-e4a4acc091b2"
@@
     )
     (path "/6861c69a-2093-46f7-addc-65485166ba0a"
-      (reference "U3") (unit 1) (value "LM3914V") (footprint "Package_LCC:PLCC-20")
-    )
-  )
+      (reference "U3") (unit 1) (value "LM3914V") (footprint "keyboard:avans-lm3914v")
+    )
+  )
